File: SUNSOFT-E301.kicad_pcb (KiCad board)
At the start: 2 copper layers, 92 x 56.7 mm, 30 parts, among them J1 Famicom Card Edge Connector, U1 HM6264, U2 FME7-5A-5B, U3 27C040, U4 27C020

Commit message: updated schematic
Parts:
- removed BT1: CR2032, custom footprints:BS-02-A1AK006
- removed C1, C4, C5, C6, C7: 0.1uF, Capacitor_SMD:C_0805_2012Metric
- removed C2, C3, C8, C9: 1uF, Capacitor_SMD:CP_Elec_4x5.3
- removed D1, D2: 1N4148, Diode_SMD:D_SOD-123
- removed JP1: SolderJumper_2_Bridged, Jumper:SolderJumper-2_P1.3mm_Bridged_RoundedPad1.0x1.5mm
- removed JP2, JP4, JP5: ~, Jumper:SolderJumper-3_P1.3mm_Open_RoundedPad1.0x1.5mm
- removed JP3: ~, Jumper:SolderJumper-2_P1.3mm_Open_RoundedPad1.0x1.5mm
- removed JP6: ~, Jumper:SolderJumper-3_P1.3mm_Bridged12_RoundedPad1.0x1.5mm
- removed R1: 1K, Resistor_SMD:R_0805_2012Metric
- removed R2: 100K, Resistor_SMD:R_0805_2012Metric
- removed R3, R4, R5: 10K, Resistor_SMD:R_0805_2012Metric
- removed Ref**: Val**, custom footprints:art_front
- removed TP1: ~, TestPoint:TestPoint_Pad_D1.0mm
- removed U1: HM6264, Package_DIP:DIP-28_W15.24mm
- removed U2: FME7-5A-5B, custom footprints:Sunsoft-5
- removed U3: 27C040, Package_DIP:DIP-32_W15.24mm_Socket
- removed U4: 27C020, Package_DIP:DIP-32_W15.24mm_Socket
Routing:
- net /CPU_R~{W}: track 116.8 -> 5.67 mm, vias 3 -> 0
- net /PRG_A15: track 80.8 -> 0.00 mm, vias 2 -> 0
- net /CHR_A15: track 78.5 -> 0.00 mm, vias 2 -> 0
- net /PRG_A16: track 75.0 -> 0.00 mm, vias 2 -> 0
- net /CHR_A17: track 71.7 -> 0.00 mm, vias 2 -> 0
- net /CHR_A10: track 73.2 -> 2.84 mm, vias 3 -> 0
- net /CPU_D7: track 72.7 -> 2.90 mm, vias 2 -> 0
- net /CPU_D6: track 70.1 -> 2.90 mm, vias 2 -> 0
- net /CHR_A12: track 64.7 -> 0.00 mm, vias 2 -> 0
- net /CPU_D5: track 65.8 -> 2.90 mm, vias 2 -> 0
- net /PRG_A17: track 61.2 -> 0.00 mm, vias 1 -> 0
- net /CPU_A14: track 63.6 -> 2.90 mm, vias 3 -> 0
- net /M2: track 63.1 -> 2.90 mm, vias 3 -> 0
- net /CPU_A9: track 63.0 -> 2.82 mm, vias 1 -> 0
- net /CPU_D0: track 62.0 -> 4.40 mm, vias 2 -> 0
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- removed copper zone on B.Cu, net /VCC_BATT
- removed copper zone on F.Cu, net /VCC_BATT
- removed copper zone on B.Cu, net GND
- removed copper zone on F.Cu, net GND
- removed copper zone on B.Cu, net Net-(C1-Pad2)
- removed copper zone on F.Cu, net Net-(C1-Pad2)
- removed copper zone on B.Cu, net VCC
- removed copper zone on F.Cu, net VCC
Other:
- board text removed: "5A/5B"
- board text removed: "BYPASS"
- board text removed: "CHR ROM 256K"
- board text removed: "EXP.AUD"
- board text removed: "FME-7"
- board text removed: "JLCJLCJLCJLC"
- board text removed: "P.18 TEST"
- board text removed: "PRG ROM 512/256 K"
- board text removed: "SRAM 8K"
- board text removed: "SS-E301 JxROM"
