File: SUNSOFT-E301.kicad_sch (KiCad schematic)
At the start: 29 parts, among them J1 Famicom Card Edge Connector, U1 HM6264, U2 FME7-5A-5B, U3 27C040, U4 27C020

Commit message: updated schematic
Parts:
- removed C4, C5, C6, C7: 0.1uF, Capacitor_SMD:C_0805_2012Metric, symbol Device:C
- removed C8, C9: 1uF, Capacitor_SMD:CP_Elec_4x5.3, symbol Device:CP1
- removed JP2, JP4, JP5: ~, Jumper:SolderJumper-3_P1.3mm_Open_RoundedPad1.0x1.5mm, symbol Jumper:SolderJumper_3_Open
- removed JP3: ~, Jumper:SolderJumper-2_P1.3mm_Open_RoundedPad1.0x1.5mm, symbol Jumper:SolderJumper_2_Open
- removed JP6: ~, Jumper:SolderJumper-3_P1.3mm_Bridged12_RoundedPad1.0x1.5mm, symbol Jumper:SolderJumper_3_Bridged12
- removed TP1: ~, TestPoint:TestPoint_Pad_D1.0mm, symbol Connector:TestPoint
- removed U2: FME7-5A-5B, custom footprints:Sunsoft-5, symbol custom_symbols:FME7-5A-5B
- removed U3: 27C040, Package_DIP:DIP-32_W15.24mm_Socket, symbol Memory_EPROM:27C040
- removed U4: 27C020, Package_DIP:DIP-32_W15.24mm_Socket, symbol Memory_EPROM:27C020
- added A1: RaspberryPi_Pico, Module_RaspberryPi_Pico:RaspberryPi_Pico_Common, symbol MCU_Module_RaspberryPi_Pico:RaspberryPi_Pico
- added U2: 27C256, Package_DIP:DIP-28_W15.24mm, symbol Memory_EPROM:27C256
Connections:
- net AUD_IN: no longer J1.45 (Pin_45), JP1.2 (B)
- net AUD_OUT: no longer J1.46 (Pin_46), JP1.1 (A)
- net CPU_A0: no longer J1.13 (Pin_13)
- net CPU_A1: no longer J1.12 (Pin_12)
- net CPU_A10: no longer J1.3 (Pin_3)
- net CPU_A11: no longer J1.2 (Pin_2)
- net CPU_A12: no longer J1.33 (Pin_33)
- net CPU_A2: no longer J1.11 (Pin_11)
- net CPU_A3: no longer J1.10 (Pin_10)
- net CPU_A4: no longer J1.9 (Pin_9)
- net CPU_A5: no longer J1.8 (Pin_8)
- net CPU_A6: no longer J1.7 (Pin_7)
- net CPU_A7: no longer J1.6 (Pin_6)
- net CPU_A8: no longer J1.5 (Pin_5)
- net CPU_A9: no longer J1.4 (Pin_4)
- net CPU_D0: no longer J1.43 (Pin_43)
- net CPU_D1: no longer J1.42 (Pin_42)
- net CPU_D2: no longer J1.41 (Pin_41)
- net CPU_D3: no longer J1.40 (Pin_40)
- net CPU_D4: no longer J1.39 (Pin_39)
- net CPU_D5: no longer J1.38 (Pin_38)
- net CPU_D6: no longer J1.37 (Pin_37)
- net CPU_D7: no longer J1.36 (Pin_36)
- net CPU_R~{W}: no longer J1.14 (Pin_14)
- net GND: now also U2.14 (GND), U2.22 (~{OE})
- net VCC: now also A1.36 (3V3), U2.1 (VPP), U2.28 (VCC)
- net ~{ROMSEL}: now also U2.20 (~{CE})
- net CHR_A10 renamed CIRAM A10
- net CPU_A13 renamed CPU A13
- net CPU_A14 renamed CPU A14
- net PPU_A0 renamed PPU A0
- net PPU_A1 renamed PPU A1
- net PPU_A10 renamed PPU A10
- net PPU_A11 renamed PPU A11
- net PPU_A12 renamed PPU A12
- net PPU_A13 renamed PPU A13
- net PPU_A2 renamed PPU A2
- net PPU_A3 renamed PPU A3
- net PPU_A4 renamed PPU A4
- net PPU_A5 renamed PPU A5
- net PPU_A6 renamed PPU A6
- net PPU_A7 renamed PPU A7
- net PPU_A8 renamed PPU A8
- net PPU_A9 renamed PPU A9
- net PPU_D0 renamed PPU D0
- net PPU_D1 renamed PPU D1
- net PPU_D2 renamed PPU D2
- net PPU_D3 renamed PPU D3
- net PPU_D4 renamed PPU D4
- net PPU_D5 renamed PPU D5
- net PPU_D6 renamed PPU D6
- net PPU_D7 renamed PPU D7
- net PPU_~{RD} renamed PPU ~{RD}
- new net: J1.45 (Pin_45), JP1.2 (B)
- new net: J1.46 (Pin_46), JP1.1 (A)
- new net: A1.13 (GND), A1.18 (GND), A1.23 (GND), A1.28 (GND), A1.3 (GND), A1.38 (GND), A1.8 (GND)
- new net CPU A0: J1.13 (Pin_13)
- new net CPU A1: J1.12 (Pin_12)
- new net CPU A10: J1.3 (Pin_3)
- new net CPU A11: J1.2 (Pin_2)
- new net CPU A12: J1.33 (Pin_33)
- new net CPU A2: J1.11 (Pin_11)
- new net CPU A3: J1.10 (Pin_10)
- new net CPU A4: J1.9 (Pin_9)
- new net CPU A5: J1.8 (Pin_8)
- new net CPU A6: J1.7 (Pin_7)
- new net CPU A7: J1.6 (Pin_6)
- new net CPU A8: J1.5 (Pin_5)
- new net CPU A9: J1.4 (Pin_4)
- new net CPU D0: J1.43 (Pin_43)
- new net CPU D1: J1.42 (Pin_42)
- new net CPU D2: J1.41 (Pin_41)
- new net CPU D3: J1.40 (Pin_40)
- new net CPU D4: J1.39 (Pin_39)
- new net CPU D5: J1.38 (Pin_38)
- new net CPU D6: J1.37 (Pin_37)
- new net CPU D7: J1.36 (Pin_36)
- new net CPU RW: J1.14 (Pin_14)
- no-connect marks 3 -> 2
Other:
- note added: "CHR ROM"
- note added: "PRG ROM"
- note removed: "CHR ROM 256K"
- note removed: "FME-7 / 5A / 5B mapper chip Bridge pads 1 and 2 of all solder jumpers if using a non-FME7 chip (5A, 5B) Otherwise, bridge pads 2 and 3 if applicable If using 512K PRG ROM, cut from VCC and bridge pads 2 and 3"
- note removed: "PRG ROM 512K/256K"
- note removed: "Pin 18 testing and debugging Keep unconnected when not in use"
- note removed: "Power filtering capacitors"
- moved on the sheet: C2, C3, JP1, R1, R2, R3

Commit message: updated schematic
Parts:
- removed U2: 27C256, Package_DIP:DIP-28_W15.24mm, symbol Memory_EPROM:27C256
- added SW1: SW_DIP_x02, symbol Switch:SW_DIP_x02
- added U2, U4: 28C256, Package_DIP:DIP-28_W15.24mm, symbol Memory_EEPROM:28C256
- added U3, U5: 27C512, Package_DIP:DIP-28_W15.24mm, symbol Memory_EPROM:27C512
Connections:
- net CPU_A0 is gone; now on net CPU A0: U1.10 (A0)
- net CPU_A1 is gone; now on net CPU A1: U1.9 (A1)
- net CPU_A10 is gone; now on net CPU A10: U1.21 (A10)
- net CPU_A11 is gone; now on net CPU A11: U1.23 (A11)
- net CPU_A2 is gone; now on net CPU A2: U1.8 (A2)
- net CPU_A3 is gone; now on net CPU A3: U1.7 (A3)
- net CPU_A4 is gone; now on net CPU A4: U1.6 (A4)
- net CPU_A5 is gone; now on net CPU A5: U1.5 (A5)
- net CPU_A6 is gone; now on net CPU A6: U1.4 (A6)
- net CPU_A7 is gone; now on net CPU A7: U1.3 (A7)
- net CPU_A8 is gone; now on net CPU A8: U1.25 (A8)
- net CPU_A9 is gone; now on net CPU A9: U1.24 (A9)
- net CPU_D0 is gone; now on net CPU D0: U1.11 (D0)
- net CPU_D1 is gone; now on net CPU D1: U1.12 (D1)
- net CPU_D2 is gone; now on net CPU D2: U1.13 (D2)
- net CPU_D3 is gone; now on net CPU D3: U1.15 (D3)
- net CPU_D4 is gone; now on net CPU D4: U1.16 (D4)
- net CPU_D5 is gone; now on net CPU D5: U1.17 (D5)
- net CPU_D6 is gone; now on net CPU D6: U1.18 (D6)
- net CPU_D7 is gone; now on net CPU D7: U1.19 (D7)
- net CPU_R~{W} is gone; now on net CPU R~{W}: U1.27 (R~{W})
- net WRAM_~{CE} is gone; now on net WRAM ~{CE}: U1.20 (~{CE})
- net AUD_IN: now also J1.45 (Pin_45), JP1.2 (B)
- net AUD_OUT: now also J1.46 (Pin_46), JP1.1 (A)
- net CPU A0: now also U2.10 (A0)
- net CPU A1: now also U2.9 (A1)
- net CPU A10: now also U2.21 (A10)
- net CPU A11: now also U2.23 (A11)
- net CPU A12: now also U2.2 (A12)
- net CPU A13: now also U2.26 (A13)
- net CPU A14: now also U2.1 (A14)
- net CPU A2: now also U2.8 (A2)
- net CPU A3: now also U2.7 (A3)
- net CPU A4: now also U2.6 (A4)
- net CPU A5: now also U2.5 (A5)
- net CPU A6: now also U2.4 (A6)
- net CPU A7: now also U2.3 (A7)
- net CPU A8: now also U2.25 (A8)
- net CPU A9: now also U2.24 (A9)
- net CPU D0: now also U2.11 (D0)
- net CPU D1: now also U2.12 (D1)
- net CPU D2: now also U2.13 (D2)
- net CPU D3: now also U2.15 (D3)
- net CPU D4: now also U2.16 (D4)
- net CPU D5: now also U2.17 (D5)
- net CPU D6: now also U2.18 (D6)
- net CPU D7: now also U2.19 (D7)
- net GND: now also U2.14 (GND), U2.22 (~{OE}), U3.14 (GND), U3.22 (~{OE}), U4.14 (GND), U4.22 (~{OE}), U5.14 (GND), U5.22 (~{OE})
- net PPU A0: now also U4.10 (A0), U4.2 (A12), U4.21 (A10), U4.23 (A11), U4.24 (A9), U4.25 (A8), U4.3 (A7), U4.4 (A6), U4.5 (A5), U4.6 (A4), U4.7 (A3), U4.8 (A2), U4.9 (A1)
- net PPU A13: now also U4.20 (~{CE})
- net PPU D0: now also U4.11 (D0)
- net PPU D1: now also U4.12 (D1)
- net PPU D2: now also U4.13 (D2)
- net PPU D3: now also U4.15 (D3)
- net PPU D4: now also U4.16 (D4)
- net PPU D5: now also U4.17 (D5)
- net PPU D6: now also U4.18 (D6)
- net PPU D7: now also U4.19 (D7)
- net VCC: now also A1.40 (VBUS), SW1.1, SW1.2, U2.27 (~{WE}), U2.28 (VCC), U3.20 (~{CE}), U4.27 (~{WE}), U4.28 (VCC), U5.20 (~{CE}); no longer A1.36 (3V3)
- net ~{IRQ}: now also A1.9 (GPIO6)
- net ~{ROMSEL}: now also U2.20 (~{CE})
- net PRG ~{CE}: now reaches A1.10 (GPIO7)
- net CHR ~{CE}: now reaches A1.11 (GPIO8)
- net WRAM ~{CE}: now reaches A1.12 (GPIO9)
- net CPU RW renamed CPU R~{W}
- net CPU_A12: no longer names the net of U1.2 (A12)
- new net EXTRA1 PWR: SW1.4, U3.28 (VCC)
- new net EXTRA2 PWR: SW1.3, U5.28 (VCC)
- no-connect marks 2 -> 4
Other:
- note added: "EXTRA ROM"
- company: Persune -> KilnApps
- title: FME-7 / 5A / 5B DevBoard (SS-E301 / JxROM) -> Pico DevBoard (UxROM)
- moved on the sheet: A1, BT1, C1, C2, C3, D1, D2, R1, R2, R3, R4, R5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
